File: flowerbot.sch (KiCad schematic (older format))
At the start: 37 parts, among them P1 CONN_01X03, P2 CONN_01X02, P3 CONN_01X03, P4 CONN_01X06, P5 USB_OTG, P6 CONN_01X03, P7 CONN_01X02, U1 LM2937_3.3V, U2 ESP-07v2, U3 CP2102

Commit message: Adding more silkscreen and sensor multiplexing.
Parts:
- removed P4: CONN_01X06, Pin_Headers:Pin_Header_Straight_1x06, symbol CONN_01X06
- removed P6: CONN_01X03, Pin_Headers:Pin_Header_Straight_1x03, symbol CONN_01X03
- added P4: CONN_01X05, Pin_Headers:Pin_Header_Straight_1x05, symbol CONN_01X05
- added U4: 74LVC1G53, Housings_SSOP:MSOP-8_3x3mm_Pitch0.65mm, symbol 74LVC1G53_Analog_MUX
Connections:
- net labels added: AMUX_SELECT
- net labels removed: IO_4
- wire segments 125 -> 134
Other:
- note added: "Sensor Probe Selector"

Commit message: Adding lots of gerber files, some new pictures, etc.
Connections:
- net +3V3: now also C4.1, P7.2 (P2), U1.3 (OUT); no longer C4.2
- net GND: now also C3.1, C4.2, U1.2 (GND); no longer C3.2, C4.1
- net at P2.1 (P1): now also C3.2, U1.1 (IN); no longer C3.1
- net CURR_PROBE renamed PROBE_SEL
- no-connect marks 22 -> 21
Other:
- moved on the sheet: C3, C4, P2, P7, U1
