File: _saved_plantb0t.sch (KiCad schematic (older format))
At the start: 34 parts, among them P1 CONN_02X09, P10 CONN_01X01, P11 CONN_01X01, P12 CONN_01X01, P2 USB_OTG, P3 CONN_02X03, Q1 BS170, SW1 SWITCH_INV, U1 ESP-12, U12 LEDx2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

Commit message: Starting routing from scratch
Parts:
- P10, P11, P12: footprint (none) -> Connect:1pin
- P13: renamed from P?; footprint (none) -> Connect:1pin
Changed lines of the file:
@@
 $EndComp
 $Comp
-L GND #PWR7
+L GND #PWR01
 U 1 1 5744B4EC
 P 2350 7450
-F 0 "#PWR7" H 2350 7200 50  0001 C CNN
+F 0 "#PWR01" H 2350 7200 50  0001 C CNN
 F 1 "GND" H 2350 7300 50  0000 C CNN
 F 2 "" H 2350 7450 50  0000 C CNN
@@
 $EndComp
 $Comp
-L GND #PWR10
+L GND #PWR02
 U 1 1 5744B5CF
 P 4400 5150
-F 0 "#PWR10" H 4400 4900 50  0001 C CNN
+F 0 "#PWR02" H 4400 4900 50  0001 C CNN
 F 1 "GND" H 4400 5000 50  0000 C CNN
 F 2 "" H 4400 5150 50  0000 C CNN
@@
 Sensor Circuits, mounts, processing and amplification
 $Comp
-L +3.3V #PWR23
+L +3.3V #PWR03
 U 1 1 57456EF8
 P 10400 5450
-F 0 "#PWR23" H 10400 5300 50  0001 C CNN
+F 0 "#PWR03" H 10400 5300 50  0001 C CNN
 F 1 "+3.3V" H 10400 5590 50  0000 C CNN
 F 2 "" H 10400 5450 50  0000 C CNN
@@
 $EndComp
 $Comp
-L GND #PWR19
+L GND #PWR04
 U 1 1 57456FFE
 P 7950 4900
-F 0 "#PWR19" H 7950 4650 50  0001 C CNN
+F 0 "#PWR04" H 7950 4650 50  0001 C CNN
 F 1 "GND" H 7950 4750 50  0000 C CNN
 F 2 "" H 7950 4900 50  0000 C CNN
@@
 Plantbus Header (Shield Extender)
 $Comp
-L +5V #PWR6
+L +5V #PWR05
 U 1 1 5745A196
 P 2350 1450
-F 0 "#PWR6" H 2350 1300 50  0001 C CNN
+F 0 "#PWR05" H 2350 1300 50  0001 C CNN
 F 1 "+5V" V 2350 1650 50  0000 C CNN
 F 2 "" H 2350 1450 50  0000 C CNN
@@
 $EndComp
 $Comp
-L GND #PWR4
+L GND #PWR06
 U 1 1 5745F516
 P 2100 5650
-F 0 "#PWR4" H 2100 5400 50  0001 C CNN
+F 0 "#PWR06" H 2100 5400 50  0001 C CNN
 F 1 "GND" H 2100 5500 50  0000 C CNN
 F 2 "" H 2100 5650 50  0000 C CNN
@@
 USB_D+
 $Comp
-L GND #PWR15
+L GND #PWR07
 U 1 1 57468586
 P 5700 5800
-F 0 "#PWR15" H 5700 5550 50  0001 C CNN
+F 0 "#PWR07" H 5700 5550 50  0001 C CNN
 F 1 "GND" H 5700 5650 50  0000 C CNN
 F 2 "" H 5700 5800 50  0000 C CNN
@@
 Temporary USB Programmer (too expensive and not properly used) \nuntil I can find something else. Very simple to set up and *should* \njust work out of the box. Found documentation online that sugested \nthat this is a working setup.
 $Comp
-L +5V #PWR21
+L +5V #PWR08
 U 1 1 5745DC51
 P 8750 3800
-F 0 "#PWR21" H 8750 3650 50  0001 C CNN
+F 0 "#PWR08" H 8750 3650 50  0001 C CNN
 F 1 "+5V" H 8750 3940 50  0000 C CNN
 F 2 "" H 8750 3800 50  0000 C CNN
@@
 $EndComp
 $Comp
-L +5V #PWR17
+L +5V #PWR09
 U 1 1 575E164D
 P 6550 4550
-F 0 "#PWR17" H 6550 4400 50  0001 C CNN
+F 0 "#PWR09" H 6550 4400 50  0001 C CNN
 F 1 "+5V" H 6550 4690 50  0000 C CNN
 F 2 "" H 6550 4550 50  0000 C CNN
@@
 Core Microcontroller
 $Comp
-L +3.3V #PWR2
+L +3.3V #PWR010
 U 1 1 575ED71A
 P 1800 4600
-F 0 "#PWR2" H 1800 4450 50  0001 C CNN
+F 0 "#PWR010" H 1800 4450 50  0001 C CNN
 F 1 "+3.3V" V 1800 4850 50  0000 C CNN
 F 2 "" H 1800 4600 50  0000 C CNN
@@
 NoConn ~ 6500 3150
 $Comp
-L GND #PWR18
+L GND #PWR011
 U 1 1 575FDBDA
 P 7700 2150
-F 0 "#PWR18" H 7700 1900 50  0001 C CNN
+F 0 "#PWR011" H 7700 1900 50  0001 C CNN
 F 1 "GND" H 7700 2000 50  0000 C CNN
 F 2 "" H 7700 2150 50  0000 C CNN
@@
 $EndComp
 $Comp
-L +5V #PWR13
+L +5V #PWR012
 U 1 1 575FE5E0
 P 5200 3800
-F 0 "#PWR13" H 5200 3650 50  0001 C CNN
+F 0 "#PWR012" H 5200 3650 50  0001 C CNN
 F 1 "+5V" H 5200 3940 50  0000 C CNN
 F 2 "" H 5200 3800 50  0000 C CNN
@@
 $EndComp
 $Comp
-L GND #PWR11
+L GND #PWR013
 U 1 1 57601863
 P 4450 3800
-F 0 "#PWR11" H 4450 3550 50  0001 C CNN
+F 0 "#PWR013" H 4450 3550 50  0001 C CNN
 F 1 "GND" H 4450 3650 50  0000 C CNN
 F 2 "" H 4450 3800 50  0000 C CNN
@@
 $EndComp
 $Comp
-L +3.3V #PWR5
+L +3.3V #PWR014
 U 1 1 57EBD05E
 P 2250 1050
-F 0 "#PWR5" H 2250 900 50  0001 C CNN
+F 0 "#PWR014" H 2250 900 50  0001 C CNN
 F 1 "+3.3V" V 2250 1200 50  0000 L CNN
 F 2 "" H 2250 1050 50  0000 C CNN
@@
 $EndComp
 $Comp
-L GND #PWR16
+L GND #PWR015
 U 1 1 57EC1675
 P 6400 7200
-F 0 "#PWR16" H 6400 6950 50  0001 C CNN
+F 0 "#PWR015" H 6400 6950 50  0001 C CNN
 F 1 "GND" H 6405 7027 50  0000 C CNN
 F 2 "" H 6400 7200 50  0000 C CNN
@@
 $EndComp
 $Comp
-L GND #PWR1
+L GND #PWR016
 U 1 1 57EC8A5F
 P 1650 2150
-F 0 "#PWR1" H 1650 1900 50  0001 C CNN
+F 0 "#PWR016" H 1650 1900 50  0001 C CNN
 F 1 "GND" H 1655 1977 50  0000 C CNN
 F 2 "" H 1650 2150 50  0000 C CNN
@@
 $EndComp
 $Comp
-L GND #PWR3
+L GND #PWR017
 U 1 1 57ECD55B
 P 1850 5350
-F 0 "#PWR3" H 1850 5100 50  0001 C CNN
+F 0 "#PWR017" H 1850 5100 50  0001 C CNN
 F 1 "GND" V 1855 5222 50  0000 R CNN
 F 2 "" H 1850 5350 50  0000 C CNN
@@
 $EndComp
 $Comp
-L +5V #PWR14
+L +5V #PWR018
 U 1 1 57ECDFEE
 P 5300 6700
-F 0 "#PWR14" H 5300 6550 50  0001 C CNN
+F 0 "#PWR018" H 5300 6550 50  0001 C CNN
 F 1 "+5V" V 5300 6900 50  0000 C CNN
 F 2 "" H 5300 6700 50  0000 C CNN
@@
 $EndComp
 $Comp
-L GND #PWR20
+L GND #PWR019
 U 1 1 57EEFB95
 P 8300 5550
-F 0 "#PWR20" H 8300 5300 50  0001 C CNN
+F 0 "#PWR019" H 8300 5300 50  0001 C CNN
 F 1 "GND" H 8300 5400 50  0000 C CNN
 F 2 "" H 8300 5550 50  0000 C CNN
@@
 NoConn ~ 6300 3150
 $Comp
-L GND #PWR22
+L GND #PWR020
 U 1 1 57EF8F73
 P 10350 1600
-F 0 "#PWR22" H 10350 1350 50  0001 C CNN
+F 0 "#PWR020" H 10350 1350 50  0001 C CNN
 F 1 "GND" H 10350 1450 50  0000 C CNN
 F 2 "" H 10350 1600 50  0000 C CNN
@@
 	1950 1650 2100 1650
 Wire Wire Line
-	2100 2050 2100 1650
-Wire Wire Line
-	1300 2050 2100 2050
+	2100 1650 2100 2050
+Wire Wire Line
+	2100 2050 1300 2050
 Wire Wire Line
 	1300 2050 1300 1850
@@
 	10100 4000 10400 4000
 $Comp
-L +3.3V #PWR8
+L +3.3V #PWR021
 U 1 1 57EF364D
 P 2650 3600
-F 0 "#PWR8" H 2650 3450 50  0001 C CNN
+F 0 "#PWR021" H 2650 3450 50  0001 C CNN
 F 1 "+3.3V" V 2650 3850 50  0000 C CNN
 F 2 "" H 2650 3600 50  0000 C CNN
@@
 $EndComp
 $Comp
-L GND #PWR9
+L GND #PWR022
 U 1 1 57EF36F4
 P 2650 3750
-F 0 "#PWR9" H 2650 3500 50  0001 C CNN
+F 0 "#PWR022" H 2650 3500 50  0001 C CNN
 F 1 "GND" V 2655 3622 50  0000 R CNN
 F 2 "" H 2650 3750 50  0000 C CNN
@@
 F 0 "P12" H 5200 1550 50  0000 C CNN
 F 1 "CONN_01X01" V 5300 1450 50  0000 C CNN
-F 2 "" H 5200 1450 50  0000 C CNN
+F 2 "Connect:1pin" H 5200 1450 50  0001 C CNN
 F 3 "" H 5200 1450 50  0000 C CNN
 	1    5200 1450
@@
 F 0 "P11" H 4900 1450 50  0000 C CNN
 F 1 "CONN_01X01" V 5000 1350 50  0000 C CNN
-F 2 "" H 4900 1350 50  0000 C CNN
+F 2 "Connect:1pin" H 4900 1350 50  0001 C CNN
 F 3 "" H 4900 1350 50  0000 C CNN
 	1    4900 1350
@@
 F 0 "P10" H 4600 1350 50  0000 C CNN
 F 1 "CONN_01X01" V 4700 1250 50  0000 C CNN
-F 2 "" H 4600 1250 50  0000 C CNN
+F 2 "Connect:1pin" H 4600 1250 50  0001 C CNN
 F 3 "" H 4600 1250 50  0000 C CNN
 	1    4600 1250
@@
 $EndComp
 $Comp
-L GND #PWR12
+L GND #PWR023
 U 1 1 580555BD
 P 5300 1000
-F 0 "#PWR12" H 5300 750 50  0001 C CNN
+F 0 "#PWR023" H 5300 750 50  0001 C CNN
 F 1 "GND" V 5300 800 50  0000 C CNN
 F 2 "" H 5300 1000 50  0000 C CNN
@@
 	5300 900  5300 1000
 $Comp
-L CONN_01X01 P?
+L CONN_01X01 P13
 U 1 1 58056575
 P 4300 1150
-F 0 "P?" H 4300 1250 50  0000 C CNN
+F 0 "P13" H 4300 1250 50  0000 C CNN
 F 1 "CONN_01X01" V 4400 1150 50  0000 C CNN
-F 2 "" H 4300 1150 50  0000 C CNN
+F 2 "Connect:1pin" H 4300 1150 50  0001 C CNN
 F 3 "" H 4300 1150 50  0000 C CNN
 	1    4300 1150
