File: plantb0t.sch (KiCad schematic (older format))
At the start: 34 parts, among them P1 CONN_02X09, P10 CONN_01X01, P11 CONN_01X01, P12 CONN_01X01, P13 CONN_01X01, P2 USB_OTG, P3 CONN_02X03, Q1 BS170, SW1 SWITCH_INV, U1 ESP-12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

Commit message: Majorly updating the board. Moving some components. Changing the Plantbot logo \o/
Parts:
- P3: footprint Pin_Headers:Pin_Header_Straight_2x03 -> base_types:prog_6pin
Changed lines of the file:
@@
 F 0 "P3" H 9650 2050 50  0000 C CNN
 F 1 "CONN_02X03" H 9650 1650 50  0000 C CNN
-F 2 "Pin_Headers:Pin_Header_Straight_2x03" H 9650 650 50  0001 C CNN
+F 2 "base_types:prog_6pin" H 9650 650 50  0001 C CNN
 F 3 "" H 9650 650 50  0000 C CNN
 	1    9650 1850
