File: plantb0t_RevA2_Sensors.sch (KiCad schematic (older format))
At the start: 24 parts

Commit message: Updating a lot of stuff...
Changed lines of the file:
@@
 LIBS:valves
 LIBS:kookie_power
-LIBS:kookie_logic
 LIBS:kookie_mcu
+LIBS:kookie_sensors
 LIBS:ESP8266
-LIBS:kookie_sensors
 LIBS:plantb0t-cache
 EELAYER 25 0
@@
 	2850 1800 2650 1800
 Wire Wire Line
-	2850 900  2850 1000
-Wire Wire Line
-	2850 1000 2850 1150
-Wire Wire Line
-	2850 1150 2850 1500
-Wire Wire Line
-	2850 1500 2850 1800
+	2850 900  2850 1800
 Wire Wire Line
 	2850 1500 2650 1500
@@
 	1600 2200 1850 2200
 Wire Wire Line
-	1600 1150 1600 1500
-Wire Wire Line
-	1600 1500 1600 2200
-Wire Wire Line
-	1600 2200 1600 2400
+	1600 1150 1600 2400
 Wire Wire Line
 	2650 1900 2950 1900
@@
 	5100 4400 5300 4400
 Wire Wire Line
-	5100 3400 5100 4200
-Wire Wire Line
-	5100 4200 5100 4300
-Wire Wire Line
-	5100 4300 5100 4400
-Wire Wire Line
-	5100 4400 5100 4550
+	5100 3400 5100 4550
 Wire Wire Line
 	5100 4300 5300 4300
@@
 	6550 1050 6900 1050
 Wire Wire Line
-	6900 1050 6900 1150
-Wire Wire Line
-	6900 1150 6900 1250
+	6900 1050 6900 1250
 Wire Wire Line
 	6650 1150 6900 1150
@@
 	6550 1900 6900 1900
 Wire Wire Line
-	6900 1900 6900 2000
-Wire Wire Line
-	6900 2000 6900 2100
+	6900 1900 6900 2100
 Wire Wire Line
 	6650 2000 6900 2000
@@
 	8350 1150 8000 1150
 Wire Wire Line
-	8000 1050 8000 1150
-Wire Wire Line
-	8000 1150 8000 1250
+	8000 1050 8000 1250
 Wire Wire Line
 	8350 1050 8000 1050
@@
 	8350 2050 8000 2050
 Wire Wire Line
-	8000 1950 8000 2050
-Wire Wire Line
-	8000 2050 8000 2150
+	8000 1950 8000 2150
 Wire Wire Line
 	8350 1950 8000 1950
@@
 	2650 5650 2650 5550
 Wire Wire Line
-	2650 6250 2650 6650
-Wire Wire Line
-	2650 6650 2650 6700
-Wire Wire Line
-	3050 5950 3200 5950
-Wire Wire Line
-	3200 5950 3300 5950
+	2650 6250 2650 6700
+Wire Wire Line
+	3050 5950 3300 5950
 Connection ~ 3200 5950
 Wire Wire Line
-	2100 6050 2300 6050
-Wire Wire Line
-	2300 6050 2450 6050
+	2100 6050 2450 6050
 Wire Wire Line
 	3200 6250 3200 5950
 Wire Wire Line
-	1850 6250 1900 6250
-Wire Wire Line
-	1900 6250 3200 6250
+	1850 6250 3200 6250
 Wire Wire Line
 	1850 6150 2100 6150
@@
 	1000 6150 1050 6150
 Wire Wire Line
-	1000 5500 1000 5750
-Wire Wire Line
-	1000 5750 1000 6150
+	1000 5500 1000 6150
 Wire Wire Line
 	1050 6250 800  6250
 Wire Wire Line
-	800  6150 800  6250
-Wire Wire Line
-	800  6250 800  6700
+	800  6150 800  6700
 Wire Wire Line
 	1950 6350 1950 6550
@@
 	2400 5850 2450 5850
 Wire Wire Line
-	8450 3600 8450 3750
-Wire Wire Line
-	8450 3750 8450 3950
+	8450 3600 8450 3950
 Wire Wire Line
 	8450 3950 9150 3950
@@
 	9150 4050 8450 4050
 Wire Wire Line
-	8450 4050 8450 4300
-Wire Wire Line
-	8450 4300 8450 4450
+	8450 4050 8450 4450
 Wire Wire Line
 	9150 4150 9100 4150
@@
 	8950 2800 10800 2800
 Wire Wire Line
-	5750 2300 5750 2350
-Wire Wire Line
-	5750 2350 5750 2400
-Wire Wire Line
-	5750 1200 5750 1700
-Wire Wire Line
-	5750 1700 5750 1900
-Wire Wire Line
-	5750 1900 5750 2000
+	5750 2300 5750 2400
+Wire Wire Line
+	5750 1200 5750 2000
 Wire Wire Line
 	5750 1700 5250 1700
@@
 	5850 3400 6300 3400
 Wire Wire Line
-	6300 3250 6300 3400
-Wire Wire Line
-	6300 3400 6300 3700
+	6300 3250 6300 3700
 Connection ~ 6300 3400
 Wire Wire Line
@@
 	6400 6200 6050 6200
 Wire Wire Line
-	6400 5600 6400 5750
-Wire Wire Line
-	6400 5750 6400 6000
-Wire Wire Line
-	6400 6000 6400 6200
+	6400 5600 6400 6200
 Wire Wire Line
 	6050 6000 6400 6000
@@
 	5050 6000 4850 6000
 Wire Wire Line
-	4850 6000 4850 6500
-Wire Wire Line
-	4850 6500 4850 6600
+	4850 6000 4850 6600
 Wire Wire Line
 	6250 6500 4850 6500
 Wire Wire Line
-	6250 6100 6250 6300
-Wire Wire Line
-	6250 6300 6250 6500
+	6250 6100 6250 6500
 Wire Wire Line
 	6250 6100 6050 6100
@@
 Connection ~ 1600 1500
 Wire Wire Line
-	1250 1000 1250 1600
-Wire Wire Line
-	1250 1600 1250 1700
+	1250 1000 1250 1700
 Wire Wire Line
 	1250 1000 2850 1000
@@
 	2250 5850 2300 5850
 Wire Wire Line
-	2300 5850 2300 6050
-Wire Wire Line
-	2300 6050 2300 6300
+	2300 5850 2300 6300
 Connection ~ 2300 6050
 $Comp

Commit message: Loading in new kookie libs
Updating Bill of Material for capacitors
Parts:
- removed C?: C, symbol C
- removed C?: CP1, symbol CP1
- removed U?: MCP3021, symbol MCP3021
- added C12: C, Capacitors_SMD:C_1206, symbol C
- C10, C11, C8: renamed from C?; footprint (none) -> Capacitors_SMD:C_1206
- gave numbers to parts that had none: 18
Connections:
- net +3V3: now also C12.2
- net GND: now also C12.1
- net SENSE_A: now also U13.15 (Y2); no longer U13.13 (Y0)
- net SENSE_C: now also U13.13 (Y0); no longer U13.15 (Y2)
- net SENSE_AMP renamed SENSE_WIRE
Other:
- note added: "Sensor Wire to MCU ADC"
- note removed: "Sensor I²C Analog Converter"

Commit message: Starting Rev A2 board routing
Parts:
- removed C9: CP1, symbol CP1
- removed U10: MCP6001, symbol MCP6001
- removed U6: PCF8574(A)T/3, symbol PCF8574(A)T/3
- added C12, C13, C9: 0.1µF, Capacitors_SMD:C_0603, symbol C
- added Q2: BS170, TO_SOT_Packages_SMD:SOT-23_Handsoldering, symbol BS170
- added R12: 10K, Resistors_SMD:R_0603, symbol R
- added R13: 100K, Resistors_SMD:R_0603, symbol R
- added U5: FXL6408, base_types:UMLP16, symbol FXL6408
- C10: renamed from C11; value C -> 0.1µF; footprint Capacitors_SMD:C_1206 -> Capacitors_SMD:C_0603
- C11: renamed from C12; value C -> 0.1µF; footprint Capacitors_SMD:C_1206 -> Capacitors_SMD:C_0603
- C7: renamed from C8; value C -> 0.1µF; footprint Capacitors_SMD:C_1206 -> Capacitors_SMD:C_0603
- C8: renamed from C10; value C -> 0.1µF; footprint Capacitors_SMD:C_1206 -> Capacitors_SMD:C_0603
- P4: renamed from P5; footprint (none) -> Pin_Headers:Pin_Header_Straight_1x02
- P5: renamed from P6; footprint (none) -> Pin_Headers:Pin_Header_Straight_1x02
- P6: renamed from P7; footprint (none) -> Pin_Headers:Pin_Header_Straight_1x02
- P7: renamed from P8; footprint (none) -> Pin_Headers:Pin_Header_Straight_1x02
- P8: renamed from P9; footprint (none) -> Pin_Headers:Pin_Header_Straight_1x04
- P9: renamed from P10; footprint (none) -> Pin_Headers:Pin_Header_Straight_1x04
- R10: renamed from R6; value R -> 100K; footprint (none) -> Resistors_SMD:R_0603
- R11: renamed from R7; footprint (none) -> Resistors_SMD:R_0603
- U10: renamed from U12; footprint (none) -> base_types:BME280
- U11: renamed from U13; footprint (none) -> Housings_SSOP:TSSOP-16_4.4x5mm_Pitch0.65mm
- U4: renamed from U5; value MCP4017 -> MCP4017 100K; footprint (none) -> TO_SOT_Packages_SMD:SC-70-6_Handsoldering
- U6: renamed from U7; footprint (none) -> base_types:sot666
- U7: renamed from U8; footprint (none) -> base_types:sot666
- U8: renamed from U9; footprint (none) -> TO_SOT_Packages_SMD:SOT-23-5
- U9: renamed from U11; footprint (none) -> TO_SOT_Packages_SMD:SOT-353
Connections:
- net +3V3: now also C9.2, Q2.1 (D), R12.1, U5.1 (~INT), U5.15 (VCC), U5.2 (V_DDIO), U5.9 (ADDR); no longer U10.8 (VDD)
- net GND: now also C12.1, C12.2, C13.2, C9.1, R13.2; no longer C8.2
- net I2C_CLOCK: now also U5.13 (SCL)
- net I2C_DATA: now also U5.14 (SDA)
- net SENABLE_A: now also U5.3 (GPIO7)
- net SENABLE_B: now also U5.4 (GPIO6)
- net SENABLE_C: now also U5.5 (GPIO5)
- net SENABLE_D: now also U5.6 (GPIO4)
- net SMUX_A: now also U5.7 (GPIO3)
- net SMUX_B: now also U5.8 (GPIO2)
- net SMUX_C: now also U5.11 (GPIO1)
- new net: C8.2, U5.16 (GND)
- new net: C13.1, U10.8 (VDD)
- new net: R12.2, U5.10 (~RST)
- new net GPIO_1: Q2.3 (S), R13.1
- new net GPIO_TRIG: Q2.2 (G), U5.12 (GPIO0)
- no-connect marks 5 -> 4
Other:
- note added: "Hirarchical Pins"
- note added: "MOSFET power gate GPIO 1"
- note removed: "Sensor Wire to MCU ADC"
- moved on the sheet: C10, C11, C8, R11, U10, U11, U4, U9

Commit message: Starting routing from scratch
Parts:
- C10, C11, C12, C13, C7, C8, C9: footprint Capacitors_SMD:C_0603 -> Capacitors_SMD:C_0805
Changed lines of the file:
@@
 $EndComp
 $Comp
-L GND #PWR023
+L GND #PWR30
 U 1 1 5744C790
 P 5100 4650
-F 0 "#PWR023" H 5100 4400 50  0001 C CNN
+F 0 "#PWR30" H 5100 4400 50  0001 C CNN
 F 1 "GND" H 5100 4500 50  0000 C CNN
 F 2 "" H 5100 4650 50  0000 C CNN
@@
 $EndComp
 $Comp
-L +3.3V #PWR024
+L +3.3V #PWR33
 U 1 1 5744C84A
 P 6300 3250
-F 0 "#PWR024" H 6300 3100 50  0001 C CNN
+F 0 "#PWR33" H 6300 3100 50  0001 C CNN
 F 1 "+3.3V" H 6300 3390 50  0000 C CNN
 F 2 "" H 6300 3250 50  0000 C CNN
@@
 SENSE_A
 $Comp
-L GND #PWR025
+L GND #PWR35
 U 1 1 5744E721
 P 7300 1250
-F 0 "#PWR025" H 7300 1000 50  0001 C CNN
+F 0 "#PWR35" H 7300 1000 50  0001 C CNN
 F 1 "GND" H 7300 1100 50  0000 C CNN
 F 2 "" H 7300 1250 50  0000 C CNN
@@
 SENSE_B
 $Comp
-L GND #PWR026
+L GND #PWR36
 U 1 1 5744E7B9
 P 7300 2100
-F 0 "#PWR026" H 7300 1850 50  0001 C CNN
+F 0 "#PWR36" H 7300 1850 50  0001 C CNN
 F 1 "GND" H 7300 1950 50  0000 C CNN
 F 2 "" H 7300 2100 50  0000 C CNN
@@
 $EndComp
 $Comp
-L GND #PWR027
+L GND #PWR37
 U 1 1 5744E95C
 P 7600 1250
-F 0 "#PWR027" H 7600 1000 50  0001 C CNN
+F 0 "#PWR37" H 7600 1000 50  0001 C CNN
 F 1 "GND" H 7600 1100 50  0000 C CNN
 F 2 "" H 7600 1250 50  0000 C CNN
@@
 SPWR_C
 $Comp
-L GND #PWR028
+L GND #PWR38
 U 1 1 5744EA2D
 P 7600 2150
-F 0 "#PWR028" H 7600 1900 50  0001 C CNN
+F 0 "#PWR38" H 7600 1900 50  0001 C CNN
 F 1 "GND" H 7600 2000 50  0000 C CNN
 F 2 "" H 7600 2150 50  0000 C CNN
@@
 SENSE_AMP
 $Comp
-L +3.3V #PWR029
+L +3.3V #PWR26
 U 1 1 5744FC44
 P 2650 5550
-F 0 "#PWR029" H 2650 5400 50  0001 C CNN
+F 0 "#PWR26" H 2650 5400 50  0001 C CNN
 F 1 "+3.3V" H 2650 5690 50  0000 C CNN
 F 2 "" H 2650 5550 50  0000 C CNN
@@
 I2C_CLOCK
 $Comp
-L +3.3V #PWR030
+L +3.3V #PWR25
 U 1 1 57450902
 P 1150 5500
-F 0 "#PWR030" H 1150 5350 50  0001 C CNN
+F 0 "#PWR25" H 1150 5350 50  0001 C CNN
 F 1 "+3.3V" H 1150 5640 50  0000 C CNN
 F 2 "" H 1150 5500 50  0000 C CNN
@@
 $EndComp
 $Comp
-L GND #PWR031
+L GND #PWR24
 U 1 1 574509BA
 P 800 6700
-F 0 "#PWR031" H 800 6450 50  0001 C CNN
+F 0 "#PWR24" H 800 6450 50  0001 C CNN
 F 1 "GND" H 800 6550 50  0000 C CNN
 F 2 "" H 800 6700 50  0000 C CNN
@@
 I²C Sense+ Extention Sockets
 $Comp
-L GND #PWR032
+L GND #PWR32
 U 1 1 57460CAA
 P 5750 2400
-F 0 "#PWR032" H 5750 2150 50  0001 C CNN
+F 0 "#PWR32" H 5750 2150 50  0001 C CNN
 F 1 "GND" H 5750 2250 50  0000 C CNN
 F 2 "" H 5750 2400 50  0000 C CNN
@@
 $EndComp
 $Comp
-L +3.3V #PWR033
+L +3.3V #PWR31
 U 1 1 574610C7
 P 5750 1200
-F 0 "#PWR033" H 5750 1050 50  0001 C CNN
+F 0 "#PWR31" H 5750 1050 50  0001 C CNN
 F 1 "+3.3V" H 5750 1340 50  0000 C CNN
 F 2 "" H 5750 1200 50  0000 C CNN
@@
 F 0 "C10" H 5725 3450 50  0000 L CNN
 F 1 "0.1µF" H 5725 3250 50  0000 L CNN
-F 2 "Capacitors_SMD:C_0603" H 5738 3200 50  0001 C CNN
+F 2 "Capacitors_SMD:C_0805" H 5738 3200 50  0001 C CNN
 F 3 "" H 5700 3350 50  0000 C CNN
 	1    5700 3350
@@
 F 0 "C8" H 3075 2300 50  0000 L CNN
 F 1 "0.1µF" H 3075 2100 50  0000 L CNN
-F 2 "Capacitors_SMD:C_0603" H 3088 2050 50  0001 C CNN
+F 2 "Capacitors_SMD:C_0805" H 3088 2050 50  0001 C CNN
 F 3 "" H 3050 2200 50  0000 C CNN
 	1    3050 2200
@@
 F 0 "C7" H 825 6100 50  0000 L CNN
 F 1 "0.1µF" H 825 5900 50  0000 L CNN
-F 2 "Capacitors_SMD:C_0603" H 838 5850 50  0001 C CNN
+F 2 "Capacitors_SMD:C_0805" H 838 5850 50  0001 C CNN
 F 3 "" H 800 6000 50  0000 C CNN
 	1    800  6000
@@
 $EndComp
 $Comp
-L +3.3V #PWR034
+L +3.3V #PWR34
 U 1 1 5746ED9B
 P 6300 5600
-F 0 "#PWR034" H 6300 5450 50  0001 C CNN
+F 0 "#PWR34" H 6300 5450 50  0001 C CNN
 F 1 "+3.3V" H 6300 5740 50  0000 C CNN
 F 2 "" H 6300 5600 50  0000 C CNN
@@
 $EndComp
 $Comp
-L GND #PWR035
+L GND #PWR29
 U 1 1 5746EEE0
 P 4800 6600
-F 0 "#PWR035" H 4800 6350 50  0001 C CNN
+F 0 "#PWR29" H 4800 6350 50  0001 C CNN
 F 1 "GND" H 4800 6450 50  0000 C CNN
 F 2 "" H 4800 6600 50  0000 C CNN
@@
 I2C_DATA
 $Comp
-L +3.3V #PWR036
+L +3.3V #PWR43
 U 1 1 57474244
 P 9650 900
-F 0 "#PWR036" H 9650 750 50  0001 C CNN
+F 0 "#PWR43" H 9650 750 50  0001 C CNN
 F 1 "+3.3V" H 9650 1040 50  0000 C CNN
 F 2 "" H 9650 900 50  0000 C CNN
@@
 $EndComp
 $Comp
-L GND #PWR037
+L GND #PWR45
 U 1 1 57474284
 P 10100 1450
-F 0 "#PWR037" H 10100 1200 50  0001 C CNN
+F 0 "#PWR45" H 10100 1200 50  0001 C CNN
 F 1 "GND" H 10100 1300 50  0000 C CNN
 F 2 "" H 10100 1450 50  0000 C CNN
@@
 I2C_DATA
 $Comp
-L +3.3V #PWR038
+L +3.3V #PWR44
 U 1 1 57474376
 P 9650 1900
-F 0 "#PWR038" H 9650 1750 50  0001 C CNN
+F 0 "#PWR44" H 9650 1750 50  0001 C CNN
 F 1 "+3.3V" H 9650 2040 50  0000 C CNN
 F 2 "" H 9650 1900 50  0000 C CNN
@@
 $EndComp
 $Comp
-L GND #PWR039
+L GND #PWR46
 U 1 1 5747437C
 P 10100 2450
-F 0 "#PWR039" H 10100 2200 50  0001 C CNN
+F 0 "#PWR46" H 10100 2200 50  0001 C CNN
 F 1 "GND" H 10100 2300 50  0000 C CNN
 F 2 "" H 10100 2450 50  0000 C CNN
@@
 OPTIONAL: Not Included in Base version
 $Comp
-L GND #PWR040
+L GND #PWR27
 U 1 1 57450ED7
 P 2650 6700
-F 0 "#PWR040" H 2650 6450 50  0001 C CNN
+F 0 "#PWR27" H 2650 6450 50  0001 C CNN
 F 1 "GND" H 2650 6550 50  0000 C CNN
 F 2 "" H 2650 6700 50  0000 C CNN
@@
 F 0 "C11" H 5775 2200 50  0000 L CNN
 F 1 "0.1µF" H 5775 2000 50  0000 L CNN
-F 2 "Capacitors_SMD:C_0603" H 5788 1950 50  0001 C CNN
+F 2 "Capacitors_SMD:C_0805" H 5788 1950 50  0001 C CNN
 F 3 "" H 5750 2100 50  0000 C CNN
 	1    5750 2100
@@
 F 0 "C9" H 5275 2200 50  0000 L CNN
 F 1 "0.1µF" H 5275 2000 50  0000 L CNN
-F 2 "Capacitors_SMD:C_0603" H 5288 1950 50  0001 C CNN
+F 2 "Capacitors_SMD:C_0805" H 5288 1950 50  0001 C CNN
 F 3 "" H 5250 2100 50  0000 C CNN
 	1    5250 2100
@@
 F 0 "C12" H 6425 6600 50  0000 L CNN
 F 1 "0.1µF" H 6425 6400 50  0000 L CNN
-F 2 "Capacitors_SMD:C_0603" H 6438 6350 50  0001 C CNN
+F 2 "Capacitors_SMD:C_0805" H 6438 6350 50  0001 C CNN
 F 3 "" H 6400 6500 50  0000 C CNN
 	1    6400 6500
@@
 F 0 "C13" H 6325 6100 50  0000 L CNN
 F 1 "0.1µF" H 6325 5900 50  0000 L CNN
-F 2 "Capacitors_SMD:C_0603" H 6338 5850 50  0001 C CNN
+F 2 "Capacitors_SMD:C_0805" H 6338 5850 50  0001 C CNN
 F 3 "" H 6300 6000 50  0000 C CNN
 	1    6300 6000
@@
 	3600 1050 3600 2200
 $Comp
-L +3.3V #PWR041
+L +3.3V #PWR28
 U 1 1 57EF0606
 P 3600 1050
-F 0 "#PWR041" H 3600 900 50  0001 C CNN
+F 0 "#PWR28" H 3600 900 50  0001 C CNN
 F 1 "+3.3V" H 3600 1190 50  0000 C CNN
 F 2 "" H 3600 1050 50  0000 C CNN
@@
 	2800 1800 2700 1800
 $Comp
-L +3.3V #PWR042
+L +3.3V #PWR39
 U 1 1 57EF1ECF
 P 8400 3350
-F 0 "#PWR042" H 8400 3200 50  0001 C CNN
+F 0 "#PWR39" H 8400 3200 50  0001 C CNN
 F 1 "+3.3V" V 8400 3600 50  0000 C CNN
 F 2 "" H 8400 3350 50  0000 C CNN
@@
 $EndComp
 $Comp
-L GND #PWR043
+L GND #PWR40
 U 1 1 57EF20B8
 P 8400 3450
-F 0 "#PWR043" H 8400 3200 50  0001 C CNN
+F 0 "#PWR40" H 8400 3200 50  0001 C CNN
 F 1 "GND" V 8400 3200 50  0000 C CNN
 F 2 "" H 8400 3450 50  0000 C CNN
@@
 	9000 4900 9400 4900
 $Comp
-L +3.3V #PWR044
+L +3.3V #PWR42
 U 1 1 57EF4EF3
 P 9150 4150
-F 0 "#PWR044" H 9150 4000 50  0001 C CNN
+F 0 "#PWR42" H 9150 4000 50  0001 C CNN
 F 1 "+3.3V" H 9150 4290 50  0000 C CNN
 F 2 "" H 9150 4150 50  0000 C CNN
@@
 $EndComp
 $Comp
-L GND #PWR045
+L GND #PWR41
 U 1 1 57EF521C
 P 8550 5050
-F 0 "#PWR045" H 8550 4800 50  0001 C CNN
+F 0 "#PWR41" H 8550 4800 50  0001 C CNN
 F 1 "GND" H 8550 4900 50  0000 C CNN
 F 2 "" H 8550 5050 50  0000 C CNN

Commit message: Correcting a wire issue around bosch sensor Finishing basic routing I²C goes through VIAS. Is that an issue?
Connections:
- net SENSOR_B is gone; now on net SENSOR_PWR: U6.4 (S2)
- net SENSOR_D is gone; now on net SENSOR_PWR: U7.4 (S2)
- net +3V3: now also C12.1, C13.1, U10.8 (VDD)
- net GND: no longer C12.1
- net SENSE_A: now also U6.6 (D1); no longer U6.1 (S1)
- net SENSE_B: now also U6.3 (D2); no longer U6.6 (D1)
- net SENSE_C: now also U7.6 (D1); no longer U7.1 (S1)
- net SENSE_D: now also U7.3 (D2); no longer U7.6 (D1)
- net SENSOR_PWR: now also U6.1 (S1), U7.1 (S1); no longer U6.3 (D2), U7.3 (D2)
Other:
- moved on the sheet: C12, C13, U10

Commit message: Majorly updating the board. Moving some components. Changing the Plantbot logo \o/
Parts:
- added P14: CONN_01X01, Connect:1pin, symbol CONN_01X01
Connections:
- net SENSE_WIRE: now also P14.1 (P1)
Changed lines of the file:
@@
 	6550 6550 6550 6450
 Connection ~ 6200 6550
+Text Label 8250 5850 2    59   ~ 0
+SENSE_AMP
+$Comp
+L CONN_01X01 P14
+U 1 1 580A7365
+P 8850 5850
+F 0 "P14" H 8850 5950 50  0000 C CNN
+F 1 "CONN_01X01" V 8950 5850 50  0000 C CNN
+F 2 "Connect:1pin" H 8850 5850 50  0001 C CNN
+F 3 "" H 8850 5850 50  0000 C CNN
+	1    8850 5850
+	1    0    0    -1
+$EndComp
+Wire Wire Line
+	8650 5850 8250 5850
 $EndSCHEMATC
