File: RevA/flowerbot.kicad_pcb (KiCad board)
At the start: 2 copper layers, 50 x 50 mm, 44 parts, among them P2 CONN_01X02, P3 CONN_01X03, P4 CONN_01X05, P5 USB_OTG, P7 CONN_01X02, U1 LM2937_3.3V, U2 ESP-07v2, U3 CP2102, U4 74LVC1G53

Commit message: Adding research material and schematics for the Rev A2 board.
Parts:
- added 112: temperature, kookie_symbols:temperature, F.Cu at (79.0, 133.9)
- added 112: Symbol_OSHW-Logo_SilkScreen, Symbols:Symbol_OSHW-Logo_SilkScreen, F.Cu at (57.5, 137.9)
- added 112: , kookie_symbols:H2O_Drop, F.Cu at (48.0, 138.4)
- added 121: temperature, kookie_symbols:temperature, F.Cu at (139.0, 73.9)
- added 121: Symbol_OSHW-Logo_SilkScreen, Symbols:Symbol_OSHW-Logo_SilkScreen, F.Cu at (117.5, 77.9)
- added 121: , kookie_symbols:H2O_Drop, F.Cu at (108.0, 78.4)
- added 122: temperature, kookie_symbols:temperature, F.Cu at (139.0, 133.9)
- added 122: Symbol_OSHW-Logo_SilkScreen, Symbols:Symbol_OSHW-Logo_SilkScreen, F.Cu at (117.5, 137.9)
- added 122: , kookie_symbols:H2O_Drop, F.Cu at (108.0, 138.4)
- added 131: temperature, kookie_symbols:temperature, F.Cu at (199.0, 73.9)
- added 131: Symbol_OSHW-Logo_SilkScreen, Symbols:Symbol_OSHW-Logo_SilkScreen, F.Cu at (177.5, 77.9)
- added 131: , kookie_symbols:H2O_Drop, F.Cu at (168.0, 78.4)
- added 132: temperature, kookie_symbols:temperature, F.Cu at (199.0, 133.9)
- added 132: Symbol_OSHW-Logo_SilkScreen, Symbols:Symbol_OSHW-Logo_SilkScreen, F.Cu at (177.5, 137.9)
- added 132: , kookie_symbols:H2O_Drop, F.Cu at (168.0, 138.4)
- added 141: temperature, kookie_symbols:temperature, F.Cu at (259.0, 73.9)
- added 141: Symbol_OSHW-Logo_SilkScreen, Symbols:Symbol_OSHW-Logo_SilkScreen, F.Cu at (237.5, 77.9)
- added 141: , kookie_symbols:H2O_Drop, F.Cu at (228.0, 78.4)
- added 142: temperature, kookie_symbols:temperature, F.Cu at (259.0, 133.9)
- added 142: Symbol_OSHW-Logo_SilkScreen, Symbols:Symbol_OSHW-Logo_SilkScreen, F.Cu at (237.5, 137.9)
- added 142: , kookie_symbols:H2O_Drop, F.Cu at (228.0, 138.4)
- added C112: 0.1µF, Capacitors_SMD:C_0603_HandSoldering, F.Cu at (72.4, 100.1)
- added C112: 0.1µF, Capacitors_SMD:C_0603_HandSoldering, F.Cu at (43.0, 132.9)
- added C112: 0.1µF, Capacitors_SMD:C_0805_HandSoldering, F.Cu at (63.0, 115.4)
- added C112: 0.1µF, Capacitors_SMD:C_0805_HandSoldering, F.Cu at (72.6, 127.9)
- added C112: C, Capacitors_SMD:C_0603_HandSoldering, F.Cu at (75.4, 113.7)
- added C112: C, Capacitors_SMD:C_0603_HandSoldering, F.Cu at (68.8, 113.9)
- added C112: 0.1µF, Capacitors_SMD:C_0603_HandSoldering, F.Cu at (68.0, 106.3)
- added C121: 0.1µF, Capacitors_SMD:C_0603_HandSoldering, F.Cu at (132.4, 40.1)
- added C121: 0.1µF, Capacitors_SMD:C_0603_HandSoldering, F.Cu at (103.0, 72.9)
- added C121: 0.1µF, Capacitors_SMD:C_0805_HandSoldering, F.Cu at (123.0, 55.4)
- added C121: 0.1µF, Capacitors_SMD:C_0805_HandSoldering, F.Cu at (132.6, 67.9)
- added C121: C, Capacitors_SMD:C_0603_HandSoldering, F.Cu at (135.4, 53.7)
- added C121: C, Capacitors_SMD:C_0603_HandSoldering, F.Cu at (128.8, 53.9)
- added C121: 0.1µF, Capacitors_SMD:C_0603_HandSoldering, F.Cu at (128.0, 46.3)
- added C122: 0.1µF, Capacitors_SMD:C_0603_HandSoldering, F.Cu at (132.4, 100.1)
- added C122: 0.1µF, Capacitors_SMD:C_0603_HandSoldering, F.Cu at (103.0, 132.9)
- added C122: 0.1µF, Capacitors_SMD:C_0805_HandSoldering, F.Cu at (123.0, 115.4)
- added C122: 0.1µF, Capacitors_SMD:C_0805_HandSoldering, F.Cu at (132.6, 127.9)
- added C122: C, Capacitors_SMD:C_0603_HandSoldering, F.Cu at (135.4, 113.7)
- added C122: C, Capacitors_SMD:C_0603_HandSoldering, F.Cu at (128.8, 113.9)
- added C122: 0.1µF, Capacitors_SMD:C_0603_HandSoldering, F.Cu at (128.0, 106.3)
- added C131: 0.1µF, Capacitors_SMD:C_0603_HandSoldering, F.Cu at (192.4, 40.1)
- added C131: 0.1µF, Capacitors_SMD:C_0603_HandSoldering, F.Cu at (163.0, 72.9)
- added C131: 0.1µF, Capacitors_SMD:C_0805_HandSoldering, F.Cu at (183.0, 55.4)
- added C131: 0.1µF, Capacitors_SMD:C_0805_HandSoldering, F.Cu at (192.6, 67.9)
- added C131: C, Capacitors_SMD:C_0603_HandSoldering, F.Cu at (195.4, 53.7)
- added C131: C, Capacitors_SMD:C_0603_HandSoldering, F.Cu at (188.8, 53.9)
- added C131: 0.1µF, Capacitors_SMD:C_0603_HandSoldering, F.Cu at (188.0, 46.3)
- added C132: 0.1µF, Capacitors_SMD:C_0603_HandSoldering, F.Cu at (192.4, 100.1)
- added C132: 0.1µF, Capacitors_SMD:C_0603_HandSoldering, F.Cu at (163.0, 132.9)
- added C132: 0.1µF, Capacitors_SMD:C_0805_HandSoldering, F.Cu at (183.0, 115.4)
- added C132: 0.1µF, Capacitors_SMD:C_0805_HandSoldering, F.Cu at (192.6, 127.9)
- added C132: C, Capacitors_SMD:C_0603_HandSoldering, F.Cu at (195.4, 113.7)
- added C132: C, Capacitors_SMD:C_0603_HandSoldering, F.Cu at (188.8, 113.9)
- added C132: 0.1µF, Capacitors_SMD:C_0603_HandSoldering, F.Cu at (188.0, 106.3)
- added C141: 0.1µF, Capacitors_SMD:C_0603_HandSoldering, F.Cu at (252.4, 40.1)
- added C141: 0.1µF, Capacitors_SMD:C_0603_HandSoldering, F.Cu at (223.0, 72.9)
- added C141: 0.1µF, Capacitors_SMD:C_0805_HandSoldering, F.Cu at (243.0, 55.4)
- added C141: 0.1µF, Capacitors_SMD:C_0805_HandSoldering, F.Cu at (252.6, 67.9)
- added C141: C, Capacitors_SMD:C_0603_HandSoldering, F.Cu at (255.4, 53.7)
- added C141: C, Capacitors_SMD:C_0603_HandSoldering, F.Cu at (248.8, 53.9)
- added C141: 0.1µF, Capacitors_SMD:C_0603_HandSoldering, F.Cu at (248.0, 46.3)
- added C142: 0.1µF, Capacitors_SMD:C_0603_HandSoldering, F.Cu at (252.4, 100.1)
- added C142: 0.1µF, Capacitors_SMD:C_0603_HandSoldering, F.Cu at (223.0, 132.9)
- added C142: 0.1µF, Capacitors_SMD:C_0805_HandSoldering, F.Cu at (243.0, 115.4)
- added C142: 0.1µF, Capacitors_SMD:C_0805_HandSoldering, F.Cu at (252.6, 127.9)
- added C142: C, Capacitors_SMD:C_0603_HandSoldering, F.Cu at (255.4, 113.7)
- added C142: C, Capacitors_SMD:C_0603_HandSoldering, F.Cu at (248.8, 113.9)
- added C142: 0.1µF, Capacitors_SMD:C_0603_HandSoldering, F.Cu at (248.0, 106.3)
- added D112: LED, LEDs:LED-0603, F.Cu at (68.8, 96.9)
- added D112: LED, LEDs:LED-0603, F.Cu at (68.9, 94.9)
- added D112: LED, LEDs:LED-0603, F.Cu at (40.3, 95.9)
- added D112: ZENER, Diodes_SMD:SOD-123, F.Cu at (80.9, 99.0)
- added D112: ZENER, Diodes_SMD:SOD-123, F.Cu at (78.6, 98.9)
- added D112: ZENER, Diodes_SMD:SOD-123, F.Cu at (76.4, 99.0)
- added D112: LED, LEDs:LED-0603, F.Cu at (67.7, 108.5)
- added D121: LED, LEDs:LED-0603, F.Cu at (128.8, 36.9)
- added D121: LED, LEDs:LED-0603, F.Cu at (128.9, 34.9)
- added D121: LED, LEDs:LED-0603, F.Cu at (100.3, 35.9)
- added D121: ZENER, Diodes_SMD:SOD-123, F.Cu at (140.9, 39.0)
- added D121: ZENER, Diodes_SMD:SOD-123, F.Cu at (138.6, 38.9)
- added D121: ZENER, Diodes_SMD:SOD-123, F.Cu at (136.4, 39.0)
- added D121: LED, LEDs:LED-0603, F.Cu at (127.7, 48.5)
- added D122: LED, LEDs:LED-0603, F.Cu at (128.8, 96.9)
- added D122: LED, LEDs:LED-0603, F.Cu at (128.9, 94.9)
- added D122: LED, LEDs:LED-0603, F.Cu at (100.3, 95.9)
- added D122: ZENER, Diodes_SMD:SOD-123, F.Cu at (140.9, 99.0)
- added D122: ZENER, Diodes_SMD:SOD-123, F.Cu at (138.6, 98.9)
- added D122: ZENER, Diodes_SMD:SOD-123, F.Cu at (136.4, 99.0)
- added D122: LED, LEDs:LED-0603, F.Cu at (127.7, 108.5)
- added D131: LED, LEDs:LED-0603, F.Cu at (188.8, 36.9)
- added D131: LED, LEDs:LED-0603, F.Cu at (188.9, 34.9)
- added D131: LED, LEDs:LED-0603, F.Cu at (160.3, 35.9)
- added D131: ZENER, Diodes_SMD:SOD-123, F.Cu at (200.9, 39.0)
- added D131: ZENER, Diodes_SMD:SOD-123, F.Cu at (198.6, 38.9)
- added D131: ZENER, Diodes_SMD:SOD-123, F.Cu at (196.4, 39.0)
- added D131: LED, LEDs:LED-0603, F.Cu at (187.7, 48.5)
- added D132: LED, LEDs:LED-0603, F.Cu at (188.8, 96.9)
- added D132: LED, LEDs:LED-0603, F.Cu at (188.9, 94.9)
- added D132: LED, LEDs:LED-0603, F.Cu at (160.3, 95.9)
- added D132: ZENER, Diodes_SMD:SOD-123, F.Cu at (200.9, 99.0)
- added D132: ZENER, Diodes_SMD:SOD-123, F.Cu at (198.6, 98.9)
- added D132: ZENER, Diodes_SMD:SOD-123, F.Cu at (196.4, 99.0)
- added D132: LED, LEDs:LED-0603, F.Cu at (187.7, 108.5)
- added D141: LED, LEDs:LED-0603, F.Cu at (248.8, 36.9)
- added D141: LED, LEDs:LED-0603, F.Cu at (248.9, 34.9)
- added D141: LED, LEDs:LED-0603, F.Cu at (220.3, 35.9)
- added D141: ZENER, Diodes_SMD:SOD-123, F.Cu at (260.9, 39.0)
- added D141: ZENER, Diodes_SMD:SOD-123, F.Cu at (258.6, 38.9)
- added D141: ZENER, Diodes_SMD:SOD-123, F.Cu at (256.4, 39.0)
- added D141: LED, LEDs:LED-0603, F.Cu at (247.7, 48.5)
- added D142: LED, LEDs:LED-0603, F.Cu at (248.8, 96.9)
- added D142: LED, LEDs:LED-0603, F.Cu at (248.9, 94.9)
- added D142: LED, LEDs:LED-0603, F.Cu at (220.3, 95.9)
- added D142: ZENER, Diodes_SMD:SOD-123, F.Cu at (260.9, 99.0)
- added D142: ZENER, Diodes_SMD:SOD-123, F.Cu at (258.6, 98.9)
- added D142: ZENER, Diodes_SMD:SOD-123, F.Cu at (256.4, 99.0)
- added D142: LED, LEDs:LED-0603, F.Cu at (247.7, 108.5)
- added G***112: LOGO, kookie_symbols:c-base, B.Cu at (79.0, 134.9)
- added G***121: LOGO, kookie_symbols:c-base, B.Cu at (139.0, 74.9)
- added G***122: LOGO, kookie_symbols:c-base, B.Cu at (139.0, 134.9)
- added G***131: LOGO, kookie_symbols:c-base, B.Cu at (199.0, 74.9)
- added G***132: LOGO, kookie_symbols:c-base, B.Cu at (199.0, 134.9)
- added G***141: LOGO, kookie_symbols:c-base, B.Cu at (259.0, 74.9)
- added G***142: LOGO, kookie_symbols:c-base, B.Cu at (259.0, 134.9)
- added I112: NXP_PSSI2021SAY, Housings_SOT-23_SOT-143_TSOT-6:SOT-23-5, F.Cu at (46.0, 132.2)
- added I112: NXP_PSSI2021SAY, Housings_SOT-23_SOT-143_TSOT-6:SOT-23-5, F.Cu at (72.5, 131.3)
- added I121: NXP_PSSI2021SAY, Housings_SOT-23_SOT-143_TSOT-6:SOT-23-5, F.Cu at (106.0, 72.2)
- added I121: NXP_PSSI2021SAY, Housings_SOT-23_SOT-143_TSOT-6:SOT-23-5, F.Cu at (132.5, 71.3)
- added I122: NXP_PSSI2021SAY, Housings_SOT-23_SOT-143_TSOT-6:SOT-23-5, F.Cu at (106.0, 132.2)
- added I122: NXP_PSSI2021SAY, Housings_SOT-23_SOT-143_TSOT-6:SOT-23-5, F.Cu at (132.5, 131.3)
- added I131: NXP_PSSI2021SAY, Housings_SOT-23_SOT-143_TSOT-6:SOT-23-5, F.Cu at (166.0, 72.2)
- added I131: NXP_PSSI2021SAY, Housings_SOT-23_SOT-143_TSOT-6:SOT-23-5, F.Cu at (192.5, 71.3)
- added I132: NXP_PSSI2021SAY, Housings_SOT-23_SOT-143_TSOT-6:SOT-23-5, F.Cu at (166.0, 132.2)
- added I132: NXP_PSSI2021SAY, Housings_SOT-23_SOT-143_TSOT-6:SOT-23-5, F.Cu at (192.5, 131.3)
- added I141: NXP_PSSI2021SAY, Housings_SOT-23_SOT-143_TSOT-6:SOT-23-5, F.Cu at (226.0, 72.2)
- added I141: NXP_PSSI2021SAY, Housings_SOT-23_SOT-143_TSOT-6:SOT-23-5, F.Cu at (252.5, 71.3)
- added I142: NXP_PSSI2021SAY, Housings_SOT-23_SOT-143_TSOT-6:SOT-23-5, F.Cu at (226.0, 132.2)
- added I142: NXP_PSSI2021SAY, Housings_SOT-23_SOT-143_TSOT-6:SOT-23-5, F.Cu at (252.5, 131.3)
- added P112: CONN_01X03, Pin_Headers:Pin_Header_Straight_1x03, F.Cu at (46.1, 121.4)
- added P112: CONN_01X05, Pin_Headers:Pin_Header_Straight_1x05, F.Cu at (39.5, 105.3)
- added P112: CONN_01X02, Pin_Headers:Pin_Header_Straight_1x02, F.Cu at (82.0, 114.7)
- added P112: CONN_01X02, Socket_Strips:Socket_Strip_Straight_1x02, F.Cu at (82.0, 120.2)
- added P112: USB_OTG, Connect:USB_Micro-B, F.Cu at (85.3, 104.4)
- added P121: CONN_01X03, Pin_Headers:Pin_Header_Straight_1x03, F.Cu at (106.2, 61.4)
- added P121: CONN_01X05, Pin_Headers:Pin_Header_Straight_1x05, F.Cu at (99.5, 45.3)
- added P121: CONN_01X02, Pin_Headers:Pin_Header_Straight_1x02, F.Cu at (142.0, 54.7)
- added P121: CONN_01X02, Socket_Strips:Socket_Strip_Straight_1x02, F.Cu at (142.0, 60.2)
- added P121: USB_OTG, Connect:USB_Micro-B, F.Cu at (145.3, 44.4)
- added P122: CONN_01X03, Pin_Headers:Pin_Header_Straight_1x03, F.Cu at (106.2, 121.4)
- added P122: CONN_01X05, Pin_Headers:Pin_Header_Straight_1x05, F.Cu at (99.5, 105.3)
- added P122: CONN_01X02, Pin_Headers:Pin_Header_Straight_1x02, F.Cu at (142.0, 114.7)
- added P122: CONN_01X02, Socket_Strips:Socket_Strip_Straight_1x02, F.Cu at (142.0, 120.2)
- added P122: USB_OTG, Connect:USB_Micro-B, F.Cu at (145.3, 104.4)
- added P131: CONN_01X03, Pin_Headers:Pin_Header_Straight_1x03, F.Cu at (166.2, 61.4)
- added P131: CONN_01X05, Pin_Headers:Pin_Header_Straight_1x05, F.Cu at (159.5, 45.3)
- added P131: CONN_01X02, Pin_Headers:Pin_Header_Straight_1x02, F.Cu at (202.0, 54.7)
- added P131: CONN_01X02, Socket_Strips:Socket_Strip_Straight_1x02, F.Cu at (202.0, 60.2)
- added P131: USB_OTG, Connect:USB_Micro-B, F.Cu at (205.3, 44.4)
- added P132: CONN_01X03, Pin_Headers:Pin_Header_Straight_1x03, F.Cu at (166.2, 121.4)
- added P132: CONN_01X05, Pin_Headers:Pin_Header_Straight_1x05, F.Cu at (159.5, 105.3)
- added P132: CONN_01X02, Pin_Headers:Pin_Header_Straight_1x02, F.Cu at (202.0, 114.7)
- added P132: CONN_01X02, Socket_Strips:Socket_Strip_Straight_1x02, F.Cu at (202.0, 120.2)
- added P132: USB_OTG, Connect:USB_Micro-B, F.Cu at (205.3, 104.4)
- added P141: CONN_01X03, Pin_Headers:Pin_Header_Straight_1x03, F.Cu at (226.2, 61.4)
- added P141: CONN_01X05, Pin_Headers:Pin_Header_Straight_1x05, F.Cu at (219.5, 45.3)
- added P141: CONN_01X02, Pin_Headers:Pin_Header_Straight_1x02, F.Cu at (262.0, 54.7)
- added P141: CONN_01X02, Socket_Strips:Socket_Strip_Straight_1x02, F.Cu at (262.0, 60.2)
- added P141: USB_OTG, Connect:USB_Micro-B, F.Cu at (265.3, 44.4)
- added P142: CONN_01X03, Pin_Headers:Pin_Header_Straight_1x03, F.Cu at (226.2, 121.4)
- added P142: CONN_01X05, Pin_Headers:Pin_Header_Straight_1x05, F.Cu at (219.5, 105.3)
- added P142: CONN_01X02, Pin_Headers:Pin_Header_Straight_1x02, F.Cu at (262.0, 114.7)
- added P142: CONN_01X02, Socket_Strips:Socket_Strip_Straight_1x02, F.Cu at (262.0, 120.2)
- added P142: USB_OTG, Connect:USB_Micro-B, F.Cu at (265.3, 104.4)
- added PROBE112: CONN_01X02, Pin_Headers:Pin_Header_Straight_1x02, F.Cu at (40.5, 137.9)
- added PROBE112: CONN_01X02, Pin_Headers:Pin_Header_Straight_1x02, F.Cu at (84.5, 137.9)
- added PROBE121: CONN_01X02, Pin_Headers:Pin_Header_Straight_1x02, F.Cu at (100.5, 77.9)
- added PROBE121: CONN_01X02, Pin_Headers:Pin_Header_Straight_1x02, F.Cu at (144.5, 77.9)
- added PROBE122: CONN_01X02, Pin_Headers:Pin_Header_Straight_1x02, F.Cu at (100.5, 137.9)
- added PROBE122: CONN_01X02, Pin_Headers:Pin_Header_Straight_1x02, F.Cu at (144.5, 137.9)
- added PROBE131: CONN_01X02, Pin_Headers:Pin_Header_Straight_1x02, F.Cu at (160.5, 77.9)
- added PROBE131: CONN_01X02, Pin_Headers:Pin_Header_Straight_1x02, F.Cu at (204.5, 77.9)
- added PROBE132: CONN_01X02, Pin_Headers:Pin_Header_Straight_1x02, F.Cu at (160.5, 137.9)
- added PROBE132: CONN_01X02, Pin_Headers:Pin_Header_Straight_1x02, F.Cu at (204.5, 137.9)
- added PROBE141: CONN_01X02, Pin_Headers:Pin_Header_Straight_1x02, F.Cu at (220.5, 77.9)
- added PROBE141: CONN_01X02, Pin_Headers:Pin_Header_Straight_1x02, F.Cu at (264.5, 77.9)
- added PROBE142: CONN_01X02, Pin_Headers:Pin_Header_Straight_1x02, F.Cu at (220.5, 137.9)
- added PROBE142: CONN_01X02, Pin_Headers:Pin_Header_Straight_1x02, F.Cu at (264.5, 137.9)
- added R112: 120, Resistors_SMD:R_0603, F.Cu at (65.9, 96.9)
- added R112: 120, Resistors_SMD:R_0603, F.Cu at (65.9, 94.9)
- added R112: 4.7k, Resistors_SMD:R_0603, F.Cu at (44.2, 127.2)
- added R112: 120, Resistors_SMD:R_0603, F.Cu at (39.1, 98.9)
- added R112: 619, Resistors_SMD:R_0603, F.Cu at (76.5, 131.3)
- added R112: 619, Resistors_SMD:R_0603, F.Cu at (48.7, 130.9)
- added R112: 4.7k, Resistors_SMD:R_0603, F.Cu at (73.5, 107.7)
- added R112: 120, Resistors_SMD:R_0603, F.Cu at (64.7, 108.5)
- added R121: 120, Resistors_SMD:R_0603, F.Cu at (125.9, 36.9)
- added R121: 120, Resistors_SMD:R_0603, F.Cu at (125.9, 34.9)
- added R121: 4.7k, Resistors_SMD:R_0603, F.Cu at (104.2, 67.2)
- added R121: 120, Resistors_SMD:R_0603, F.Cu at (99.1, 38.9)
- added R121: 619, Resistors_SMD:R_0603, F.Cu at (136.5, 71.3)
- added R121: 619, Resistors_SMD:R_0603, F.Cu at (108.7, 70.9)
- added R121: 4.7k, Resistors_SMD:R_0603, F.Cu at (133.5, 47.7)
- added R121: 120, Resistors_SMD:R_0603, F.Cu at (124.7, 48.5)
- added R122: 120, Resistors_SMD:R_0603, F.Cu at (125.9, 96.9)
- added R122: 120, Resistors_SMD:R_0603, F.Cu at (125.9, 94.9)
- added R122: 4.7k, Resistors_SMD:R_0603, F.Cu at (104.2, 127.2)
- added R122: 120, Resistors_SMD:R_0603, F.Cu at (99.1, 98.9)
- added R122: 619, Resistors_SMD:R_0603, F.Cu at (136.5, 131.3)
- added R122: 619, Resistors_SMD:R_0603, F.Cu at (108.7, 130.9)
- added R122: 4.7k, Resistors_SMD:R_0603, F.Cu at (133.5, 107.7)
- added R122: 120, Resistors_SMD:R_0603, F.Cu at (124.7, 108.5)
- added R131: 120, Resistors_SMD:R_0603, F.Cu at (185.9, 36.9)
- added R131: 120, Resistors_SMD:R_0603, F.Cu at (185.9, 34.9)
- added R131: 4.7k, Resistors_SMD:R_0603, F.Cu at (164.2, 67.2)
- added R131: 120, Resistors_SMD:R_0603, F.Cu at (159.1, 38.9)
- added R131: 619, Resistors_SMD:R_0603, F.Cu at (196.5, 71.3)
- added R131: 619, Resistors_SMD:R_0603, F.Cu at (168.7, 70.9)
- added R131: 4.7k, Resistors_SMD:R_0603, F.Cu at (193.5, 47.7)
- added R131: 120, Resistors_SMD:R_0603, F.Cu at (184.7, 48.5)
- added R132: 120, Resistors_SMD:R_0603, F.Cu at (185.9, 96.9)
- added R132: 120, Resistors_SMD:R_0603, F.Cu at (185.9, 94.9)
- added R132: 4.7k, Resistors_SMD:R_0603, F.Cu at (164.2, 127.2)
- added R132: 120, Resistors_SMD:R_0603, F.Cu at (159.1, 98.9)
- added R132: 619, Resistors_SMD:R_0603, F.Cu at (196.5, 131.3)
- added R132: 619, Resistors_SMD:R_0603, F.Cu at (168.7, 130.9)
- added R132: 4.7k, Resistors_SMD:R_0603, F.Cu at (193.5, 107.7)
- added R132: 120, Resistors_SMD:R_0603, F.Cu at (184.7, 108.5)
- added R141: 120, Resistors_SMD:R_0603, F.Cu at (245.9, 36.9)
- added R141: 120, Resistors_SMD:R_0603, F.Cu at (245.9, 34.9)
- added R141: 4.7k, Resistors_SMD:R_0603, F.Cu at (224.2, 67.2)
- added R141: 120, Resistors_SMD:R_0603, F.Cu at (219.1, 38.9)
- added R141: 619, Resistors_SMD:R_0603, F.Cu at (256.5, 71.3)
- added R141: 619, Resistors_SMD:R_0603, F.Cu at (228.7, 70.9)
- added R141: 4.7k, Resistors_SMD:R_0603, F.Cu at (253.5, 47.7)
- added R141: 120, Resistors_SMD:R_0603, F.Cu at (244.7, 48.5)
- added R142: 120, Resistors_SMD:R_0603, F.Cu at (245.9, 96.9)
- added R142: 120, Resistors_SMD:R_0603, F.Cu at (245.9, 94.9)
- added R142: 4.7k, Resistors_SMD:R_0603, F.Cu at (224.2, 127.2)
- added R142: 120, Resistors_SMD:R_0603, F.Cu at (219.1, 98.9)
- added R142: 619, Resistors_SMD:R_0603, F.Cu at (256.5, 131.3)
- added R142: 619, Resistors_SMD:R_0603, F.Cu at (228.7, 130.9)
- added R142: 4.7k, Resistors_SMD:R_0603, F.Cu at (253.5, 107.7)
- added R142: 120, Resistors_SMD:R_0603, F.Cu at (244.7, 108.5)
- added REF**112: gnd_hole_2.25mm, kookie_utilities:gnd_hole_2.25mm, F.Cu at (40.5, 133.2)
- added REF**112: gnd_hole_2.25mm, kookie_utilities:gnd_hole_2.25mm, F.Cu at (84.5, 133.2)
- added REF**112: gnd_hole_2.25mm, kookie_utilities:gnd_hole_2.25mm, F.Cu at (85.5, 94.9)
- added REF**121: gnd_hole_2.25mm, kookie_utilities:gnd_hole_2.25mm, F.Cu at (100.5, 73.2)
- added REF**121: gnd_hole_2.25mm, kookie_utilities:gnd_hole_2.25mm, F.Cu at (144.5, 73.2)
- added REF**121: gnd_hole_2.25mm, kookie_utilities:gnd_hole_2.25mm, F.Cu at (145.5, 34.9)
- added REF**122: gnd_hole_2.25mm, kookie_utilities:gnd_hole_2.25mm, F.Cu at (100.5, 133.2)
- added REF**122: gnd_hole_2.25mm, kookie_utilities:gnd_hole_2.25mm, F.Cu at (144.5, 133.2)
- added REF**122: gnd_hole_2.25mm, kookie_utilities:gnd_hole_2.25mm, F.Cu at (145.5, 94.9)
- added REF**131: gnd_hole_2.25mm, kookie_utilities:gnd_hole_2.25mm, F.Cu at (160.5, 73.2)
- added REF**131: gnd_hole_2.25mm, kookie_utilities:gnd_hole_2.25mm, F.Cu at (204.5, 73.2)
- added REF**131: gnd_hole_2.25mm, kookie_utilities:gnd_hole_2.25mm, F.Cu at (205.5, 34.9)
- added REF**132: gnd_hole_2.25mm, kookie_utilities:gnd_hole_2.25mm, F.Cu at (160.5, 133.2)
- added REF**132: gnd_hole_2.25mm, kookie_utilities:gnd_hole_2.25mm, F.Cu at (204.5, 133.2)
- added REF**132: gnd_hole_2.25mm, kookie_utilities:gnd_hole_2.25mm, F.Cu at (205.5, 94.9)
- added REF**141: gnd_hole_2.25mm, kookie_utilities:gnd_hole_2.25mm, F.Cu at (220.5, 73.2)
- added REF**141: gnd_hole_2.25mm, kookie_utilities:gnd_hole_2.25mm, F.Cu at (264.5, 73.2)
- added REF**141: gnd_hole_2.25mm, kookie_utilities:gnd_hole_2.25mm, F.Cu at (265.5, 34.9)
- added REF**142: gnd_hole_2.25mm, kookie_utilities:gnd_hole_2.25mm, F.Cu at (220.5, 133.2)
- added REF**142: gnd_hole_2.25mm, kookie_utilities:gnd_hole_2.25mm, F.Cu at (264.5, 133.2)
- added REF**142: gnd_hole_2.25mm, kookie_utilities:gnd_hole_2.25mm, F.Cu at (265.5, 94.9)
- added RESET112: SW_BTN, kookie_utilities:SW_TACTILE_SHALLOW, F.Cu at (57.2, 122.1)
- added RESET121: SW_BTN, kookie_utilities:SW_TACTILE_SHALLOW, F.Cu at (117.2, 62.1)
- added RESET122: SW_BTN, kookie_utilities:SW_TACTILE_SHALLOW, F.Cu at (117.2, 122.1)
- added RESET131: SW_BTN, kookie_utilities:SW_TACTILE_SHALLOW, F.Cu at (177.2, 62.1)
- added RESET132: SW_BTN, kookie_utilities:SW_TACTILE_SHALLOW, F.Cu at (177.2, 122.1)
- added RESET141: SW_BTN, kookie_utilities:SW_TACTILE_SHALLOW, F.Cu at (237.2, 62.1)
- added RESET142: SW_BTN, kookie_utilities:SW_TACTILE_SHALLOW, F.Cu at (237.2, 122.1)
- added Temp Probe112: CONN_01X03, Socket_Strips:Socket_Strip_Straight_1x03, F.Cu at (69.2, 136.2)
- added Temp Probe121: CONN_01X03, Socket_Strips:Socket_Strip_Straight_1x03, F.Cu at (129.2, 76.2)
- added Temp Probe122: CONN_01X03, Socket_Strips:Socket_Strip_Straight_1x03, F.Cu at (129.2, 136.2)
- added Temp Probe131: CONN_01X03, Socket_Strips:Socket_Strip_Straight_1x03, F.Cu at (189.2, 76.2)
- added Temp Probe132: CONN_01X03, Socket_Strips:Socket_Strip_Straight_1x03, F.Cu at (189.2, 136.2)
- added Temp Probe141: CONN_01X03, Socket_Strips:Socket_Strip_Straight_1x03, F.Cu at (249.2, 76.2)
- added Temp Probe142: CONN_01X03, Socket_Strips:Socket_Strip_Straight_1x03, F.Cu at (249.2, 136.2)
- added U112: CP2102, Housings_DFN_QFN:QFN-28-1EP_5x5mm_Pitch0.5mm, F.Cu at (67.8, 101.4)
- added U112: ESP-07v2, ESP8266:ESP-07v2, F.Cu at (44.7, 102.6)
- added U112: LM2937_3.3V, Housings_SOT-89:SOT89-3_Housing, F.Cu at (72.1, 114.0)
- added U112: 74LVC1G53, Housings_SSOP:MSOP-8_3x3mm_Pitch0.65mm, F.Cu at (57.5, 130.9)
- added U121: CP2102, Housings_DFN_QFN:QFN-28-1EP_5x5mm_Pitch0.5mm, F.Cu at (127.8, 41.4)
- added U121: ESP-07v2, ESP8266:ESP-07v2, F.Cu at (104.7, 42.6)
- added U121: LM2937_3.3V, Housings_SOT-89:SOT89-3_Housing, F.Cu at (132.1, 54.0)
- added U121: 74LVC1G53, Housings_SSOP:MSOP-8_3x3mm_Pitch0.65mm, F.Cu at (117.5, 70.9)
- added U122: CP2102, Housings_DFN_QFN:QFN-28-1EP_5x5mm_Pitch0.5mm, F.Cu at (127.8, 101.4)
- added U122: ESP-07v2, ESP8266:ESP-07v2, F.Cu at (104.7, 102.6)
- added U122: LM2937_3.3V, Housings_SOT-89:SOT89-3_Housing, F.Cu at (132.1, 114.0)
- added U122: 74LVC1G53, Housings_SSOP:MSOP-8_3x3mm_Pitch0.65mm, F.Cu at (117.5, 130.9)
- added U131: CP2102, Housings_DFN_QFN:QFN-28-1EP_5x5mm_Pitch0.5mm, F.Cu at (187.8, 41.4)
- added U131: ESP-07v2, ESP8266:ESP-07v2, F.Cu at (164.7, 42.6)
- added U131: LM2937_3.3V, Housings_SOT-89:SOT89-3_Housing, F.Cu at (192.1, 54.0)
- added U131: 74LVC1G53, Housings_SSOP:MSOP-8_3x3mm_Pitch0.65mm, F.Cu at (177.5, 70.9)
- added U132: CP2102, Housings_DFN_QFN:QFN-28-1EP_5x5mm_Pitch0.5mm, F.Cu at (187.8, 101.4)
- added U132: ESP-07v2, ESP8266:ESP-07v2, F.Cu at (164.7, 102.6)
- added U132: LM2937_3.3V, Housings_SOT-89:SOT89-3_Housing, F.Cu at (192.1, 114.0)
- added U132: 74LVC1G53, Housings_SSOP:MSOP-8_3x3mm_Pitch0.65mm, F.Cu at (177.5, 130.9)
- added U141: CP2102, Housings_DFN_QFN:QFN-28-1EP_5x5mm_Pitch0.5mm, F.Cu at (247.8, 41.4)
- added U141: ESP-07v2, ESP8266:ESP-07v2, F.Cu at (224.7, 42.6)
- added U141: LM2937_3.3V, Housings_SOT-89:SOT89-3_Housing, F.Cu at (252.1, 54.0)
- added U141: 74LVC1G53, Housings_SSOP:MSOP-8_3x3mm_Pitch0.65mm, F.Cu at (237.5, 70.9)
- added U142: CP2102, Housings_DFN_QFN:QFN-28-1EP_5x5mm_Pitch0.5mm, F.Cu at (247.8, 101.4)
- added U142: ESP-07v2, ESP8266:ESP-07v2, F.Cu at (224.7, 102.6)
- added U142: LM2937_3.3V, Housings_SOT-89:SOT89-3_Housing, F.Cu at (252.1, 114.0)
- added U142: 74LVC1G53, Housings_SSOP:MSOP-8_3x3mm_Pitch0.65mm, F.Cu at (237.5, 130.9)
- Temp Probe111: renamed from Temp Probe
- moved D111 113.8 mm to (68.8, 36.9)
- moved 111 113.8 mm to (79.0, 73.9)
- moved 111 113.8 mm to (48.0, 78.4)
- moved C111 113.8 mm to (72.6, 67.9)
- moved C111 113.8 mm to (63.0, 55.4)
- moved C111 113.8 mm to (43.0, 72.9)
- moved C111 113.8 mm to (68.0, 46.3)
- moved D111 113.8 mm to (68.9, 34.9)
- moved D111 113.8 mm to (40.3, 35.9)
- moved D111 113.8 mm to (76.4, 39.0)
- moved D111 113.8 mm to (80.9, 39.0)
- moved D111 113.8 mm to (78.6, 38.9)
- moved G***111 113.8 mm to (79.0, 74.9)
- moved I111 113.8 mm to (46.0, 72.2)
- moved P111 113.8 mm to (46.1, 61.4)
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- gave numbers to parts that had none: 1
- renumbered C1 to C111, C2 to C111, C5 to C111, C6 to C111, C7 to C111, C3 to C111, C4 to C111, D1 to D111, D2 to D111, D3 to D111, D4 to D111, D5 to D111, D6 to D111, D7 to D111, G*** to G***111, I1 to I111, I2 to I111, P3 to P111, P5 to P111, P7 to P111, P2 to P111, P4 to P111, PROBE1 to PROBE111, PROBE2 to PROBE111, R1 to R111, R2 to R111, R3 to R111, R4 to R111, R5 to R111, R6 to R111, R7 to R111, R8 to R111, REF** to REF**111, RESET1 to RESET111, U3 to U111, U1 to U111, U2 to U111, U4 to U111
Routing:
- net GND: track 149.2 -> 1193.3 mm, vias 1 -> 8
- net +3V3: track 133.3 -> 1066.0 mm, vias 2 -> 16
- net /RES: track 49.8 -> 398.3 mm
- net /AMUX_SELECT: track 37.6 -> 300.9 mm, vias 2 -> 16
- net /PROBE_SEL: track 36.6 -> 293.0 mm, vias 1 -> 8
- net +5V: track 34.5 -> 276.0 mm
- net /H2O_PROBE: track 31.3 -> 250.6 mm
- net /IO_13: track 27.8 -> 222.1 mm
- net Net-(D6-Pad1): track 24.5 -> 196.4 mm, vias 2 -> 16
- net Net-(D7-Pad1): track 22.7 -> 181.7 mm, vias 2 -> 16
- net /RX_D: track 22.6 -> 181.0 mm
- net /IO_5: track 19.6 -> 157.1 mm
- net /CH_PD: track 17.0 -> 136.1 mm
- net /TEMP_PROBE: track 16.7 -> 133.7 mm
- net /TX_D: track 16.1 -> 128.6 mm
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Other:
- board size 50 x 50 mm -> 245 x 130 mm
