File: plantb0t/plantb0t.sch (KiCad schematic (older format))
At the start: 34 parts, among them P1 CONN_02X09, P10 CONN_01X01, P11 CONN_01X01, P12 CONN_01X01, P13 CONN_01X01, P2 USB_OTG, P3 CONN_02X03, Q1 BS170, SW1 SWITCH_INV, U1 ESP-12, U12 LEDx2, U2 CP2102, U3 ZXCL5213V30H5CT-ND

Commit message: Updating a bunch of project files to the state that went into production on 2017-01-01
Parts:
- removed C2: 1µF, Capacitors_SMD:C_0805, symbol C
- removed C3: 0.1µF, Capacitors_SMD:C_0805, symbol C
- removed C4: 4.7µF, Capacitors_SMD:c_elec_4x5.3, symbol CP1
- removed D5, D6, D7: Zener, Diodes_SMD:SOD-323, symbol ZENERsmall
- removed P2: USB_OTG, Connect:USB_Micro-B, symbol USB_OTG
- removed P3: CONN_02X03, base_types:prog_6pin, symbol CONN_02X03
- removed R6: 4.7k, Resistors_SMD:R_0603, symbol R
- removed U12: LEDx2, base_types:SML-52, symbol LEDx2
- removed U2: CP2102, Housings_DFN_QFN:QFN-28-1EP_5x5mm_Pitch0.5mm, symbol CP2102
- removed U3: ZXCL5213V30H5CT-ND, TO_SOT_Packages_SMD:SOT-23-5, symbol ZXCL5213V30H5CT-ND
- added P6: CONN_01X04, Socket_Strips:Socket_Strip_Straight_1x04, symbol CONN_01X04
- added U2: LED_x2, kookie_sml:SML-521, symbol LED_x2
- added U3: ZXCL5213, TO_SOT_Packages_SMD:SOT-23-5, symbol ZXCL5213
- C1: footprint Capacitors_SMD:c_elec_4x5.3 -> Capacitors_SMD:c_elec_4x4.5
- C3: renamed from C6; footprint Capacitors_SMD:c_elec_4x5.3 -> Capacitors_SMD:c_elec_4x4.5
- D1: symbol LED -> LED-RESCUE-plantb0t
- D2: renamed from D3; symbol LED -> LED-RESCUE-plantb0t
- D3: renamed from D4; symbol LED -> LED-RESCUE-plantb0t
- P1: footprint Pin_Headers:Pin_Header_Straight_2x09 -> Socket_Strips:Socket_Strip_Straight_2x09
- SW1: footprint Buttons_Switches_SMD:SW_SPST_B3U-3100P-B -> base_types:SSAJ120100
- renumbered C5 to C2, P13 to P2, P10 to P3, P11 to P4, P12 to P5, R7 to R6, R8 to R7, R9 to R8
Connections:
- net labels removed: SLEEP_ST, USB_D+, USB_D-
- wire segments 165 -> 117
- no-connect marks 20 -> 0
Other:
- note added: "Grounded screw holes"
- note added: "Hier könnte Ihre Werbung stehen!"
- note added: "UART programming & Power"
- note removed: "For consumer variant the big USB programmer won't be present. \nDo initial programming of the ESP by connecting temporary programming\nheader. USB programmer can be retrofit. This does not affect \nUSB power or protection diodes on VCC/ 5V."
- note removed: "Ghettogrammer"
- note removed: "Temporary USB Programmer (too expensive and not properly used) \nuntil I can find something else. Very simple to set up and *should* \njust work out of the box. Found documentation online that sugested \nthat this is a working setup."
- note removed: "USB Port & USB Power"
- moved on the sheet: C2, C3, Q1, R3, R8
