File: plantb0t/plantb0t_RevA2_Sensors.sch (KiCad schematic (older format))
At the start: 27 parts, among them P14 CONN_01X01, P4 CONN_01X02, P5 CONN_01X02, P6 CONN_01X02, P7 CONN_01X02, P8 CONN_01X04, P9 CONN_01X04, Q2 BS170, U10 BMP280, U11 74HC(T)4051, U4 MCP4017 100K, U5 FXL6408, U6 FC6946010R, U7 FC6946010R, U8 MCP6001, U9 PSSI2021SAY

Commit message: Updating a bunch of project files to the state that went into production on 2017-01-01
Parts:
- removed U5: FXL6408, base_types:UMLP16, symbol FXL6408
- added C6: 0.1µF, Capacitors_SMD:C_0805, symbol C
- added P14: CONN_01X01, base_types:1pin-SMD, symbol CONN_01X01
- added U5: XRA1220(P), Housings_SSOP:TSSOP-16_4.4x5mm_Pitch0.65mm, symbol XRA1220(P)
- P10: renamed from P7; footprint Pin_Headers:Pin_Header_Straight_1x02 -> Socket_Strips:Socket_Strip_Straight_1x02
- P11: renamed from P14; footprint Connect:1pin -> base_types:1pin-SMD
- P12: renamed from P8; footprint Pin_Headers:Pin_Header_Straight_1x04 -> Socket_Strips:Socket_Strip_Straight_1x04
- P13: renamed from P9; footprint Pin_Headers:Pin_Header_Straight_1x04 -> Socket_Strips:Socket_Strip_Straight_1x04
- P7: renamed from P4; footprint Pin_Headers:Pin_Header_Straight_1x02 -> Socket_Strips:Socket_Strip_Straight_1x02
- P8: renamed from P5; footprint Pin_Headers:Pin_Header_Straight_1x02 -> Socket_Strips:Socket_Strip_Straight_1x02
- P9: renamed from P6; footprint Pin_Headers:Pin_Header_Straight_1x02 -> Socket_Strips:Socket_Strip_Straight_1x02
- renumbered C12 to C10, C13 to C11, C7 to C4, C8 to C5, C9 to C7, C10 to C8, C11 to C9, R12 to R10, R13 to R12, R10 to R9
Connections:
- wire segments 156 -> 162
Other:
- moved on the sheet: C4, C5, C7, P13, R10, R9, U10, U4, U8

Commit message: Moving documentation over to fodt. Adding a bunch of stuff. Merging to master because yolo
Parts:
- R10: value 10K -> 220
- R11: value R -> 220
- U8: symbol MCP6001 -> MCP6001-RESCUE-plantb0t
Changed lines of the file:
@@
 LIBS:valves
 LIBS:kookie_regulators
-LIBS:kookie_passive
 LIBS:kookie_nxp
 LIBS:kookie_microchip
 LIBS:kookie_iox
-LIBS:kookie_bosch
 LIBS:ESP8266
-LIBS:kookie_74xx
 LIBS:plantb0t-cache
-EELAYER 25 0
+EELAYER 26 0
 EELAYER END
 $Descr A4 11693 8268
@@
 MUXED_SENSE
 $Comp
-L MCP6001 U8
+L MCP6001-RESCUE-plantb0t U8
 U 1 1 5744F5D1
 P 2800 5950
@@
 P 5500 1550
 F 0 "R11" V 5580 1550 50  0000 C CNN
-F 1 "R" V 5500 1550 50  0000 C CNN
+F 1 "220" V 5500 1550 50  0000 C CNN
 F 2 "Resistors_SMD:R_0603" V 5430 1550 50  0001 C CNN
 F 3 "" H 5500 1550 50  0000 C CNN
@@
 P 3300 1500
 F 0 "R10" V 3200 1500 50  0000 C CNN
-F 1 "10K" V 3300 1500 50  0000 C CNN
+F 1 "220" V 3300 1500 50  0000 C CNN
 F 2 "Resistors_SMD:R_0603" V 3230 1500 50  0001 C CNN
 F 3 "" H 3300 1500 50  0000 C CNN
