File: plantbot_core/plantbot_core.kicad_pcb (KiCad board)
At the start: 2 copper layers, 50 x 50 mm, 55 parts, among them P1 CONN_02X09, P10 CONN_01X02, P11 CONN_01X01, P12 CONN_01X04, P13 CONN_01X04, P14 CONN_01X01, P2 CONN_01X01, P3 CONN_01X01, P4 CONN_01X01, P5 CONN_01X01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

Commit message: Fixing some KiCad issues (I think)
Routing:
- net GND: track 92.0 -> 90.5 mm
Changed lines of the file:
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@@
-(kicad_pcb (version 4) (host pcbnew 4.0.5)
+(kicad_pcb (version 4) (host pcbnew 4.0.7)
   (general
     (links 153)
@@
     (thickness 1.6)
     (drawings 65)
-    (tracks 711)
+    (tracks 709)
     (zones 0)
     (modules 55)
@@
     (effects (font (size 0.6 0.6) (thickness 0.125)))
   )
-  (gr_text GND (at 134.15 112.75 360) (layer F.SilkS)
+  (gr_text GND (at 134.15 112.75) (layer F.SilkS)
     (effects (font (size 0.6 0.6) (thickness 0.125)))
   )
@@
   (via (at 142.7 96.125) (size 0.6) (drill 0.4) (layers F.Cu B.Cu) (net 2))
   (segment (start 143.125 96.55) (end 142.7 96.125) (width 0.25) (layer F.Cu) (net 2))
-  (segment (start 157.375 101.6) (end 157.375 103.025) (width 0.25) (layer F.Cu) (net 2))
-  (segment (start 157.375 103.025) (end 157.35 103.05) (width 0.25) (layer F.Cu) (net 2))
   (segment (start 157.595 106.495) (end 158.195 106.495) (width 0.25) (layer F.Cu) (net 2))
   (segment (start 143.125 98.05) (end 143.125 97.125) (width 0.25) (layer F.Cu) (net 2))
