File: plantbot_core/plantbot_core.sch (KiCad schematic (older format))
At the start: 25 parts, among them P1 CONN_02X09, P2 CONN_01X01, P3 CONN_01X01, P4 CONN_01X01, P5 CONN_01X01, P6 CONN_01X04, Q1 BS170, SW1 SWITCH_INV, U1 ESP-12, U2 LED_x2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

Commit message: Fixing some KiCad issues (I think)
Parts:
- Q1: symbol BS170 -> BS170-RESCUE-plantbot_core
Changed lines of the file:
@@
 EESchema Schematic File Version 2
-LIBS:plantb0t-rescue
+LIBS:plantbot_core-rescue
 LIBS:power
 LIBS:device
@@
 LIBS:contrib
 LIBS:valves
+LIBS:ESP8266
+LIBS:kookie_iox
+LIBS:kookie_microchip
+LIBS:kookie_nxp
 LIBS:kookie_regulators
-LIBS:kookie_nxp
-LIBS:kookie_microchip
-LIBS:kookie_iox
-LIBS:ESP8266
-LIBS:plantb0t-cache
-EELAYER 26 0
+LIBS:plantbot_core-cache
+EELAYER 25 0
 EELAYER END
 $Descr A4 11693 8268
@@
 U 5744BD50
 F0 "Sensor Mounts" 59
-F1 "plantb0t_RevA2_Sensors.sch" 39
+F1 "plantbot_core_RevA2_Sensors.sch" 39
 F2 "I2C_DATA" I R 2250 3000 79
 F3 "I2C_CLOCK" I R 2250 3150 79
@@
 $EndComp
 $Comp
-L BS170 Q1
+L BS170-RESCUE-plantbot_core Q1
 U 1 1 57456A48
 P 10300 5150
