File: plantbot_core/plantbot_core_RevA2_Sensors.sch (KiCad schematic (older format))
At the start: 29 parts, among them P10 CONN_01X02, P11 CONN_01X01, P12 CONN_01X04, P13 CONN_01X04, P14 CONN_01X01, P7 CONN_01X02, P8 CONN_01X02, P9 CONN_01X02, Q2 BS170, U10 BMP280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

Commit message: Fixing some KiCad issues (I think)
Parts:
- Q2: symbol BS170 -> BS170-RESCUE-plantbot_core
Changed lines of the file:
@@
 EESchema Schematic File Version 2
-LIBS:plantb0t-rescue
+LIBS:plantbot_core-rescue
 LIBS:power
 LIBS:device
@@
 LIBS:contrib
 LIBS:valves
+LIBS:ESP8266
+LIBS:kookie_iox
+LIBS:kookie_microchip
+LIBS:kookie_nxp
 LIBS:kookie_regulators
-LIBS:kookie_nxp
-LIBS:kookie_microchip
-LIBS:kookie_iox
-LIBS:ESP8266
-LIBS:plantb0t-cache
-EELAYER 26 0
+LIBS:plantbot_core-cache
+EELAYER 25 0
 EELAYER END
 $Descr A4 11693 8268
@@
 GPIO_1
 $Comp
-L BS170 Q2
+L BS170-RESCUE-plantbot_core Q2
 U 1 1 57EF4D65
 P 9050 4450
